File: r3/src/safeproject-mic-r3.kicad_sch (KiCad schematic)
At the start: 23 parts, among them J101 2842142-4, U101 PCMD3180

Commit message: Add fiducials. Change text, move to mask layer.
Parts:
- added FID1, FID2: Fiducial, Fiducial:Fiducial_0.5mm_Mask1mm, symbol Mechanical:Fiducial
Changed lines of the file:
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@@
     (pin "1")
+  )
+  (symbol (lib_id "Mechanical:Fiducial") (at 220.98 147.32 0) (unit 1)
+    (in_bom yes) (on_board yes) (fields_autoplaced)
+    (property "Reference" "FID1" (id 0) (at 223.52 146.6849 0)
+      (effects (font (size 1.27 1.27)) (justify left))
+    )
+    (property "Value" "Fiducial" (id 1) (at 223.52 149.2249 0)
+      (effects (font (size 1.27 1.27)) (justify left))
+    )
+    (property "Footprint" "Fiducial:Fiducial_0.5mm_Mask1mm" (id 2) (at 220.98 147.32 0)
+      (effects (font (size 1.27 1.27)) hide)
+    )
+    (property "Datasheet" "~" (id 3) (at 220.98 147.32 0)
+      (effects (font (size 1.27 1.27)) hide)
+    )
+  )
+  (symbol (lib_id "Mechanical:Fiducial") (at 220.98 153.67 0) (unit 1)
+    (in_bom yes) (on_board yes) (fields_autoplaced)
+    (property "Reference" "FID2" (id 0) (at 223.52 153.0349 0)
+      (effects (font (size 1.27 1.27)) (justify left))
+    )
+    (property "Value" "Fiducial" (id 1) (at 223.52 155.5749 0)
+      (effects (font (size 1.27 1.27)) (justify left))
+    )
+    (property "Footprint" "Fiducial:Fiducial_0.5mm_Mask1mm" (id 2) (at 220.98 153.67 0)
+      (effects (font (size 1.27 1.27)) hide)
+    )
+    (property "Datasheet" "~" (id 3) (at 220.98 153.67 0)
+      (effects (font (size 1.27 1.27)) hide)
+    )
   )
   (symbol (lib_id "Device:R_Small") (at 82.55 74.93 90) (unit 1)
@@
       (reference "C112") (unit 1) (value "1uF") (footprint "Capacitor_SMD:C_0603_1608Metric")
     )
+    (path "/a788886d-d09e-4d57-adf9-1c25b7f0fa6a"
+      (reference "FID1") (unit 1) (value "Fiducial") (footprint "Fiducial:Fiducial_0.5mm_Mask1mm")
+    )
+    (path "/eafa243e-34f8-4b07-b653-9ee6d7cb3e7a"
+      (reference "FID2") (unit 1) (value "Fiducial") (footprint "Fiducial:Fiducial_0.5mm_Mask1mm")
+    )
     (path "/e981660f-7717-449b-8d64-17301d3e16cd"

Commit message: Connect Wurth spacer mounting pads to GND
Parts:
- H101, H102: footprint jeffmakes-footprints:wurth-spacer-WA-SMSI-9774070360R -> Mounting_Wuerth:Mounting_Wuerth_WA-SMSI-M3_H7mm_9774070360; symbol Mechanical:MountingHole -> Mechanical:MountingHole_Pad
- renumbered TP101 to TP1, TP102 to TP2, TP103 to TP3
Connections:
- net GND: now also H101.1, H102.1
Changed lines of the file:
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@@
   (symbol (lib_id "Connector:TestPoint") (at 90.17 74.93 0) (unit 1)
     (in_bom yes) (on_board yes)
-    (property "Reference" "TP102" (id 0) (at 92.71 71.12 0)
+    (property "Reference" "TP2" (id 0) (at 92.71 71.12 0)
       (effects (font (size 1.27 1.27)) (justify left))
     )
@@
   (symbol (lib_id "Connector:TestPoint") (at 90.17 83.82 0) (unit 1)
     (in_bom yes) (on_board yes)
-    (property "Reference" "TP103" (id 0) (at 92.71 80.01 0)
+    (property "Reference" "TP3" (id 0) (at 92.71 80.01 0)
       (effects (font (size 1.27 1.27)) (justify left))
     )
@@
   (symbol (lib_id "Connector:TestPoint") (at 180.34 125.73 270) (unit 1)
     (in_bom yes) (on_board yes)
-    (property "Reference" "TP101" (id 0) (at 185.42 124.46 90)
+    (property "Reference" "TP1" (id 0) (at 185.42 124.46 90)
       (effects (font (size 1.27 1.27)) (justify left))
     )
@@
     )
     (property "Datasheet" "" (id 3) (at 195.58 72.39 0)
+      (effects (font (size 1.27 1.27)) hide)
+    )
+    (pin "1")
+  )
+  (symbol (lib_id "power:GND") (at 220.98 127.635 0) (mirror y) (unit 1)
+    (in_bom yes) (on_board yes)
+    (property "Reference" "#PWR0120" (id 0) (at 220.98 133.985 0)
+      (effects (font (size 1.27 1.27)) hide)
+    )
+    (property "Value" "GND" (id 1) (at 220.98 131.445 0))
+    (property "Footprint" "" (id 2) (at 220.98 127.635 0)
+      (effects (font (size 1.27 1.27)) hide)
+    )
+    (property "Datasheet" "" (id 3) (at 220.98 127.635 0)
+      (effects (font (size 1.27 1.27)) hide)
+    )
+    (pin "1")
+  )
+  (symbol (lib_id "power:GND") (at 220.98 139.065 0) (mirror y) (unit 1)
+    (in_bom yes) (on_board yes)
+    (property "Reference" "#PWR0119" (id 0) (at 220.98 145.415 0)
+      (effects (font (size 1.27 1.27)) hide)
+    )
+    (property "Value" "GND" (id 1) (at 220.98 142.875 0))
+    (property "Footprint" "" (id 2) (at 220.98 139.065 0)
+      (effects (font (size 1.27 1.27)) hide)
+    )
+    (property "Datasheet" "" (id 3) (at 220.98 139.065 0)
       (effects (font (size 1.27 1.27)) hide)
     )
@@
     (pin "2")
   )
-  (symbol (lib_id "Mechanical:MountingHole") (at 220.98 129.54 0) (unit 1)
-    (in_bom yes) (on_board yes)
-    (property "Reference" "H101" (id 0) (at 224.79 128.9049 0)
-      (effects (font (size 1.27 1.27)) (justify left))
-    )
-    (property "Value" "wurth-spacer-WA-SMSI-9774070360" (id 1) (at 224.79 131.4449 0)
-      (effects (font (size 1.27 1.27)) (justify left))
-    )
-    (property "Footprint" "jeffmakes-footprints:wurth-spacer-WA-SMSI-9774070360R" (id 2) (at 220.98 129.54 0)
-      (effects (font (size 1.27 1.27)) hide)
-    )
-    (property "Datasheet" "~" (id 3) (at 220.98 129.54 0)
-      (effects (font (size 1.27 1.27)) hide)
-    )
-  )
-  (symbol (lib_id "Mechanical:MountingHole") (at 220.98 137.16 0) (unit 1)
-    (in_bom yes) (on_board yes)
-    (property "Reference" "H102" (id 0) (at 224.79 136.5249 0)
-      (effects (font (size 1.27 1.27)) (justify left))
-    )
-    (property "Value" "wurth-spacer-WA-SMSI-9774070360" (id 1) (at 224.79 139.0649 0)
-      (effects (font (size 1.27 1.27)) (justify left))
-    )
-    (property "Footprint" "jeffmakes-footprints:wurth-spacer-WA-SMSI-9774070360R" (id 2) (at 220.98 137.16 0)
-      (effects (font (size 1.27 1.27)) hide)
-    )
-    (property "Datasheet" "~" (id 3) (at 220.98 137.16 0))
-  )
   (symbol (lib_id "Device:C_Small") (at 63.5 59.69 90) (unit 1)
     (in_bom yes) (on_board yes)
@@
     (pin "1")
     (pin "2")
+  )
+  (symbol (lib_id "Mechanical:MountingHole_Pad") (at 220.98 125.095 0) (unit 1)
+    (in_bom yes) (on_board yes)
+    (property "Reference" "H101" (id 0) (at 224.79 124.4599 0)
+      (effects (font (size 1.27 1.27)) (justify left))
+    )
+    (property "Value" "wurth-spacer-WA-SMSI-9774070360" (id 1) (at 224.79 126.9999 0)
+      (effects (font (size 1.27 1.27)) (justify left))
+    )
+    (property "Footprint" "Mounting_Wuerth:Mounting_Wuerth_WA-SMSI-M3_H7mm_9774070360" (id 2) (at 220.98 125.095 0)
+      (effects (font (size 1.27 1.27)) hide)
+    )
+    (property "Datasheet" "~" (id 3) (at 220.98 125.095 0)
+      (effects (font (size 1.27 1.27)) hide)
+    )
+    (pin "1")
+  )
+  (symbol (lib_id "Mechanical:MountingHole_Pad") (at 220.98 136.525 0) (unit 1)
+    (in_bom yes) (on_board yes)
+    (property "Reference" "H102" (id 0) (at 224.79 135.8899 0)
+      (effects (font (size 1.27 1.27)) (justify left))
+    )
+    (property "Value" "wurth-spacer-WA-SMSI-9774070360" (id 1) (at 224.79 138.4299 0)
+      (effects (font (size 1.27 1.27)) (justify left))
+    )
+    (property "Footprint" "Mounting_Wuerth:Mounting_Wuerth_WA-SMSI-M3_H7mm_9774070360" (id 2) (at 220.98 136.525 0)
+      (effects (font (size 1.27 1.27)) hide)
+    )
+    (property "Datasheet" "~" (id 3) (at 220.98 136.525 0)
+      (effects (font (size 1.27 1.27)) hide)
+    )
+    (pin "1")
   )
   (symbol (lib_id "Connector_Generic:Conn_02x04_Odd_Even") (at 234.95 99.06 0) (unit 1)
@@
       (reference "#PWR0118") (unit 1) (value "+3V3") (footprint "")
     )
+    (path "/73eb6a0c-8f8c-46dd-815d-d2c83d21e3d4"
+      (reference "#PWR0119") (unit 1) (value "GND") (footprint "")
+    )
+    (path "/40df3846-ccbe-4354-838a-6830af32a312"
+      (reference "#PWR0120") (unit 1) (value "GND") (footprint "")
+    )
     (path "/b5693a0b-6f55-4a5d-88a7-9cf0f294a4e2"
       (reference "C101") (unit 1) (value "100nF") (footprint "Capacitor_SMD:C_0402_1005Metric")
@@
     )
     (path "/e981660f-7717-449b-8d64-17301d3e16cd"
-      (reference "H101") (unit 1) (value "wurth-spacer-WA-SMSI-9774070360") (footprint "jeffmakes-footprints:wurth-spacer-WA-SMSI-9774070360R")
+      (reference "H101") (unit 1) (value "wurth-spacer-WA-SMSI-9774070360") (footprint "Mounting_Wuerth:Mounting_Wuerth_WA-SMSI-M3_H7mm_9774070360")
     )
     (path "/5775c3a6-8e4d-46b6-8692-e3035ff2dff7"
-      (reference "H102") (unit 1) (value "wurth-spacer-WA-SMSI-9774070360") (footprint "jeffmakes-footprints:wurth-spacer-WA-SMSI-9774070360R")
+      (reference "H102") (unit 1) (value "wurth-spacer-WA-SMSI-9774070360") (footprint "Mounting_Wuerth:Mounting_Wuerth_WA-SMSI-M3_H7mm_9774070360")
     )
     (path "/cfddb752-5d42-40a4-a784-47604c60f145"
@@
     )
     (path "/619f3b9b-1e8c-450e-9e99-81a019399861"
-      (reference "TP101") (unit 1) (value "TestPoint") (footprint "TestPoint:TestPoint_Pad_D1.0mm")
+      (reference "TP1") (unit 1) (value "TestPoint") (footprint "TestPoint:TestPoint_Pad_D1.0mm")
     )
     (path "/4b39f222-8e62-4663-996d-2300900cb879"
-      (reference "TP102") (unit 1) (value "TestPoint") (footprint "TestPoint:TestPoint_Pad_D1.0mm")
+      (reference "TP2") (unit 1) (value "TestPoint") (footprint "TestPoint:TestPoint_Pad_D1.0mm")
     )
     (path "/3da0f188-afb1-44d5-84b4-254947699d98"
-      (reference "TP103") (unit 1) (value "TestPoint") (footprint "TestPoint:TestPoint_Pad_D1.0mm")
+      (reference "TP3") (unit 1) (value "TestPoint") (footprint "TestPoint:TestPoint_Pad_D1.0mm")
     )
     (path "/bb961c22-975d-43a9-ac2a-7246f1939233"

Commit message: Shorten test point names
Parts:
- renumbered TP1 to TP101, TP2 to TP102, TP3 to TP103
Changed lines of the file:
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@@
   (symbol (lib_id "Connector:TestPoint") (at 90.17 74.93 0) (unit 1)
     (in_bom yes) (on_board yes)
-    (property "Reference" "TP2" (id 0) (at 92.71 71.12 0)
+    (property "Reference" "TP102" (id 0) (at 92.71 71.12 0)
       (effects (font (size 1.27 1.27)) (justify left))
     )
@@
   (symbol (lib_id "Connector:TestPoint") (at 90.17 83.82 0) (unit 1)
     (in_bom yes) (on_board yes)
-    (property "Reference" "TP3" (id 0) (at 92.71 80.01 0)
+    (property "Reference" "TP103" (id 0) (at 92.71 80.01 0)
       (effects (font (size 1.27 1.27)) (justify left))
     )
@@
   (symbol (lib_id "Connector:TestPoint") (at 180.34 125.73 270) (unit 1)
     (in_bom yes) (on_board yes)
-    (property "Reference" "TP1" (id 0) (at 185.42 124.46 90)
+    (property "Reference" "TP101" (id 0) (at 185.42 124.46 90)
       (effects (font (size 1.27 1.27)) (justify left))
     )
@@
     )
     (path "/619f3b9b-1e8c-450e-9e99-81a019399861"
-      (reference "TP1") (unit 1) (value "TestPoint") (footprint "TestPoint:TestPoint_Pad_D1.0mm")
+      (reference "TP101") (unit 1) (value "TestPoint") (footprint "TestPoint:TestPoint_Pad_D1.0mm")
     )
     (path "/4b39f222-8e62-4663-996d-2300900cb879"
-      (reference "TP2") (unit 1) (value "TestPoint") (footprint "TestPoint:TestPoint_Pad_D1.0mm")
+      (reference "TP102") (unit 1) (value "TestPoint") (footprint "TestPoint:TestPoint_Pad_D1.0mm")
     )
     (path "/3da0f188-afb1-44d5-84b4-254947699d98"
-      (reference "TP3") (unit 1) (value "TestPoint") (footprint "TestPoint:TestPoint_Pad_D1.0mm")
+      (reference "TP103") (unit 1) (value "TestPoint") (footprint "TestPoint:TestPoint_Pad_D1.0mm")
     )
     (path "/bb961c22-975d-43a9-ac2a-7246f1939233"
