File: r5/src/bugg-mic-r5.kicad_sch (KiCad schematic)
At the start: 25 parts, among them J301 2842142-4, U301 PCMD3180

Commit message: Replace 0603 resistor with 0402
Parts:
- R303: footprint Resistor_SMD:R_0603_1608Metric -> Resistor_SMD:R_0402_1005Metric
Changed lines of the file:
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@@
       (effects (font (size 1.27 1.27)) (justify right))
     )
-    (property "Footprint" "Resistor_SMD:R_0603_1608Metric" (at 195.58 62.23 0)
+    (property "Footprint" "Resistor_SMD:R_0402_1005Metric" (at 195.58 62.23 0)
       (effects (font (size 1.27 1.27)) hide)
     )

Commit message: Replace board-to-board header with type with alignment pegs
Parts:
- J301: footprint jeffmakes-footprints:PinHeader_2x04_P2.00mm_Vertical_SMD_AMPMODU -> jeffmakes-footprints:xPRN042MAMP-RC
Changed lines of the file:
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@@
       (effects (font (size 1.27 1.27)) (justify left))
     )
-    (property "Footprint" "jeffmakes-footprints:PinHeader_2x04_P2.00mm_Vertical_SMD_AMPMODU" (at 234.95 99.06 0)
+    (property "Footprint" "jeffmakes-footprints:xPRN042MAMP-RC" (at 234.95 99.06 0)
       (effects (font (size 1.27 1.27)) hide)
     )

Commit message: Fabrication data exported with lacKi
Parts:
- C301, C305, C307, C309, C311: Voltage (none) -> 50V
- J301: value 2842142-4 -> NRPN042MAMS-RC; Digikey (none) -> S6009-04-ND; MPN (none) -> NRPN042MAMS-RC; Manufacturer (none) -> Sullins
- MIC301: Digikey (none) -> SPH0641LU4H-1; MPN (none) -> SPH0641LU4H-1; Manufacturer (none) -> Knowles; Mouser (none) -> 721-SPH0641LU4H-1
- SP301, SP302: Digikey (none) -> 732-5274-1-ND; MPN (none) -> 9774070360R; Manufacturer (none) -> Wurth; Mouser (none) -> 710-9774070360R
- U301: Digikey (none) -> 296-PCMD3180IRTWTDKR-ND; MPN (none) -> PCMD3180IRTWT; Manufacturer (none) -> TI; Mouser (none) -> 595-PCMD3180IRTWT
